Commit message: Add 3D LiDAR model to Turtlebot4

File: src/robot_nav_ws/src/turtlebot4/turtlebot4_description/urdf/standard/turtlebot4.urdf.xacro (robot description, xacro)
@@ -9,4 +9,5 @@
   <xacro:include filename="$(find turtlebot4_description)/urdf/standard/tower_sensor_plate.urdf.xacro" />
   <xacro:include filename="$(find turtlebot4_description)/urdf/standard/weight_block.urdf.xacro" />
+  <xacro:include filename="$(find turtlebot4_description)/urdf/sensors/lidar3d.urdf.xacro" />
   <!-- Mechanical properties -->
   <xacro:property name="shell_z_offset"                value="${3*cm2m}" />
@@ -33,4 +34,8 @@
   <xacro:property name="oakd_pro_y_offset"             value="${0*cm2m}"/>
   <xacro:property name="oakd_pro_z_offset"             value="${9.676*cm2m}"/>
+  <!-- Add a new property for the LiDAR mounting position -->
+  <xacro:property name="lidar_x_offset" value="0.0"/>
+  <xacro:property name="lidar_y_offset" value="0.0"/>
+  <xacro:property name="lidar_z_offset" value="${30.0*cm2m}"/> <!-- about 30cm above ground -->
   <joint name="shell_link_joint" type="fixed">
     <parent link="base_link"/>
@@ -101,3 +106,6 @@
     <origin xyz="${oakd_pro_x_offset} ${oakd_pro_y_offset} ${oakd_pro_z_offset}"/>
   </xacro:oakd>
+  <xacro:lidar3d name="lidar3d" parent_link="shell_link" gazebo="$(arg gazebo)">
+    <origin xyz="${lidar_x_offset} ${lidar_y_offset} ${lidar_z_offset}" rpy="0 0 0"/>
+  </xacro:lidar3d>
 </robot>
